File: kikit_stuff/board.kicad_pcb (KiCad board)
At the start: 2 copper layers, 17.8 x 24.2 mm, 18 parts, among them J1 Conn_01x01_Pin, J10 Conn_01x05, J2 Conn_01x01_Pin, J3 Conn_01x01_Pin, J4 Conn_01x01_Pin, J5 Conn_01x01_Pin, J6 Conn_01x01_Pin, J8 Conn_01x01, J9 Conn_01x01, SW1 Switch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

Commit message: added gerbers
Parts:
- removed the G*** at (119.9, 92.5) (x2)
- removed the G*** at (129.4, 82.9) (x2)
- removed the G*** at (121.3, 85.2) (x2)
- added G*** (x2): LOGO, GraphicsKicad:signature_small, F.Cu at (129.5, 83.0)
- added G*** (x2): LOGO, GraphicsKicad:snake, F.Cu at (120.0, 92.5)
- added G*** (x2): LOGO, GraphicsKicad:signature, B.Cu at (121.3, 85.1)
Routing:
- net GND: vias 1 -> 2
- added copper zone on B.Cu, net GND
- added copper zone on F.Cu, net GND
